Commit message: folders

File: ugv_ws/src/my_ugv_description/urdf/ugv.urdf.xacro (robot description, xacro)
@@ -11,5 +11,5 @@
             <origin xyz="0.15 0 0.075"/>
             <geometry>
-                <box size="0.3 0.3 0.15"/>
+                <mesh filename="package://my_ugv_description/meshes/ugv_chassis.stl" />
             </geometry>
             <material name="white">
